File: RUTH_balance_bot/2026_12_2Wheel_Balance_Robot_v1.kicad_pcb (KiCad board)
At the start: 2 copper layers, 68.6 x 53.4 mm, 56 parts, among them J1 Conn_01x04, J2 CONN_MPU6050, J3 USB_C_Receptacle_USB2.0_14P, J4 ESP_Conn, J5 BATT_CONN, J6 M1_CONN, J7 M2_CONN, J8 ENCODER_CONN, J9 MT6701_CONN, SW2 SW_uP_Reset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

Commit message: main
Parts:
- moved C3 1.75 mm to (135.8, 79.1)
Routing:
- net +3.3V: track 87.4 -> 206.0 mm, vias 2 -> 22
- net +5V: track 20.3 -> 102.6 mm
- net VM: track 0.00 -> 53.4 mm, vias 0 -> 6
- net 5V_REG: track 0.00 -> 23.6 mm
- net Net-(D5-A): track 0.00 -> 12.0 mm, vias 0 -> 2
- net GND: track 73.0 -> 83.5 mm, vias 49 -> 53
- net Net-(D3-A): track 0.00 -> 2.26 mm
- net (no net): vias 1 -> 0
Other:
- board text added: "Nicolas Ruth Embedded Systems Project 5/5/26"
